File: Hardware/IoT-Based-Smart-Aquarium-Monitor-&-Control-System.kicad_pcb (KiCad board)
At the start: 2 copper layers, 75 parts, among them J1 Screw_Terminal_01x03, J10 TDS_Sensor, J11 12V JACK, J12 Screw_Terminal_01x03, J13 FISH_FEEDER01x03_SMotor, J13PSW1 12V JACK, J14 BMS, J15 S Panel, J16 12V JACK, J17 240V_JACK_Out, J18 240V__Jack_In, J19 Stress-free_lighting, J2 12V JACK, J20 Heat Dissipation Unit, J21 Conn_01x08, J22 (RTC), J3 Buck Converter, J4 Screw_Terminal_01x03, J5 LCD 22(SCL) 21(SDA), J6 BUZZER, J7 pH_SENSOR, J8 Turbidity_SENSOR, J9 TEM SENSOR, K4 SANYOU_SRD_Form_C, K5 SANYOU_SRD_Form_C, K6 SANYOU_SRD_Form_C, Q1 BC547, Q2 BC547, Q3 BC547, Q4 BC547, SW1 SW_Push

Commit message: feat: enhance licensing, security, and project documentation
- Implement multi-license model (MIT, CERN-OHL-S-2.0, CC BY 4.0)
- Secure firmware credentials with secrets.example.h and .gitignore
- Update README with professional badges, star buttons, and synchronized voice specifications
- Finalize hardware design, Gerber files, and BOM
Other:
- board text added: "License: CERN-OHL-S-2.0"
- board text removed: "License: MIT License"
Changed lines of the file:
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@@
 		(comment 1 "Module: Fundamentals of Computing (IT1140) - Y1S1")
 		(comment 2 "Designed by: Sachin Rathnayaka (WRSCN)")
-		(comment 3 "License: MIT License")
+		(comment 3 "License: CERN-OHL-S-2.0")
 		(comment 4 "Repo: github.com/SachinRathnayaka/Smart-Aquarium-Monitor-Control-System")
 		(comment 5 "Sheet Name: Main")
@@
 			(drillshape 0)
 			(scaleselection 1)
-			(outputdirectory "Gerber_Files/")
+			(outputdirectory "Gerber_Files/new gerber/")
 		)
 	)
@@
 		)
 	)
-	(gr_text "License: MIT License"
+	(gr_text "License: CERN-OHL-S-2.0"
 		(locked yes)
 		(at 162.79 76.95 0)
@@
 		)
 	)
-	(gr_text "License: MIT License"
+	(gr_text "License: CERN-OHL-S-2.0"
 		(locked yes)
-		(at 168.14 93.17 0)
+		(at 169.3 93.17 0)
 		(layer "B.Cu")
 		(effects
@@
 	)
 	(zone
+		(locked yes)
 		(layer "B.Cu")
 		(hatch edge 0.5)
